Commit message: Update kobuki.urdf.xacro

File: cartographer_ros/cartographer_ros/launch/includes/urdf/kobuki.urdf.xacro (robot description, xacro)
@@ -30,5 +30,5 @@
         <geometry>
           <!-- new mesh -->
-          <mesh filename="package:/cartographer_ros/launch/includes/meshes/main_body.dae" />
+          <mesh filename="package://cartographer_ros/launch/includes/meshes/main_body.dae" />
         </geometry>
         <origin xyz="0.001 0 0.05199" rpy="0 0 0"/>
@@ -65,5 +65,5 @@
       <visual>
         <geometry>
-          <mesh filename="package:/cartographer_ros/launch/includes/meshes/wheel.dae"/>
+          <mesh filename="package://cartographer_ros/launch/includes/meshes/wheel.dae"/>
         </geometry>
         <origin xyz="0 0 0" rpy="0 0 0"/>
@@ -92,5 +92,5 @@
       <visual>
         <geometry>
-          <mesh filename="package:/cartographer_ros/launch/includes/meshes/wheel.dae"/>
+          <mesh filename="package://cartographer_ros/launch/includes/meshes/wheel.dae"/>
         </geometry>
         <origin xyz="0 0 0" rpy="0 0 0"/>
@@ -223,5 +223,5 @@
       <origin xyz="0 0 0" rpy="0 0 0"/>
       <geometry>
-        <mesh filename="package:/cartographer_ros/launch/includes/meshes/hokuyo.dae"/>
+        <mesh filename="package://cartographer_ros/launch/includes/meshes/hokuyo.dae"/>
       </geometry>
     </visual>
